Commit message: spr limity/ urdf?

File: zad3/urdf/move.urdf (robot description, URDF)
Before this commit: robot my_robot, 4 links, 3 joints
Joints:
- joint base_to_link1: limit (none) -> lower=-3.1415 upper=3.1415 effort=1000.0 velocity=0.5
- joint link1_to_link2: limit lower=-1.57075 upper=1.57075 effort=1000.0 velocity=0.5 -> lower=-3.1415 upper=3.1415 effort=1000.0 velocity=0.5
- joint link2_to_link3: limit (none) -> lower=-0.3 upper=0.3 effort=1000.0 velocity=0.5

Commit message: some fixs with dh/urdf/rviz

File: zad3/urdf/move.urdf (robot description, URDF)
Before this commit: robot my_robot, 4 links, 3 joints
Links:
- link base_link: geometry visual cylinder length=0.7 radius=0.2
- link link_3: geometry visual cylinder length=0.5 radius=0.04
Joints:
- joint base_to_link1: type continuous -> revolute
- joint link1_to_link2: limit lower=-3.1415 upper=3.1415 effort=1000.0 velocity=0.5 -> lower=-1.57 upper=1.57 effort=1000.0 velocity=0.5
- joint link2_to_link3: limit lower=-0.3 upper=0.3 effort=1000.0 velocity=0.5 -> lower=-0.03 upper=0.45 effort=1000.0 velocity=0.5; type fixed -> prismatic

Commit message: last fixs work good with limits

File: zad3/urdf/move.urdf (robot description, URDF)
Before this commit: robot my_robot, 4 links, 3 joints
Joints:
- removed joint link2_to_link3
- added joint link2_link3: type prismatic, parent link_2, child link_3, origin xyz=${props['i3']['j_xyz']} rpy=${props['i3']['j_rpy']}, axis 0 0 1, limit lower=-0.03 upper=0.25 effort=1000.0 velocity=0.5
